File: hardware/circuit_boards/base_pwr/BaSe_PWR_V4_0.kicad_sch (KiCad schematic)
At the start: 111 parts, among them J1 12VDC In, J1 USB_C_Receptacle, J11 MOTOR, J12 Conn_01x04_Socket, J13 HPH1-A-16-UA, J2 HRS-1B-16-GA, J3 USB3_A, J3 USB_B_Micro, J4 Conn_01x07_Pin, J6 Conn_02x06_Odd_Even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

Commit message: [HW] add bill of materials
Parts:
- C5, C7: Digikey Part Number (none) -> 732-7672-1-ND; SPN 732-7672-1-ND -> (none); SPR Digikey -> (none)
- D1: Digikey Part Number (none) -> 732-9949-1-ND; SPN 732-9949-1-ND -> (none); SPR Digikey -> (none)
- D3: Digikey SK34-TPMSCT-ND -> (none); Digikey Part Number (none) -> SK34-TPMSCT-ND
- D4: Digikey Part Number (none) -> SK64L-TPMSCT-ND; SPN SK64L-TPMSCT-ND -> (none)
- D5, D6, D7, D8: Digikey Part Number (none) -> 1N4148WRHGCT-ND; SPN 1N4148WRHGCT-ND -> (none)
- F1: Digikey Part Number (none) -> F3147CT-ND; Irated 5A -> (none); digikey F3147CT-ND -> (none)
- FFC_Cable1: Digikey WM16429-ND -> (none); Digikey Part Number (none) -> WM16429-ND; SPN WM16429-ND -> (none); SPR Digikey -> (none)
- FL1: Digikey Part Number (none) -> 240-2502-1-ND; SPN 240-2502-1-ND -> (none)
- J1, J3: Digikey Part Number (none) -> 137-RAHPCUC31AU1TRCT-ND
- J13: Digikey Part Number (none) -> HPH1-A-16-UA; SPN HPH1-A-16-UA -> (none)
- J14: Digikey Part Number (none) -> WM10954CT-ND; SPN WM10954CT-ND -> (none)
- J2: Digikey Part Number (none) -> HRS-1B-16-GA; SPN HRS-1B-16-GA -> (none)
- J7: Digikey 664-GSB343K331HRCT-ND -> (none); Digikey Part Number (none) -> 664-GSB343K331HRCT-ND
- K1, K2: Digikey Part Number (none) -> 399-11031-5-ND; SPN 399-11031-5-ND -> (none); SPR Digikey -> (none)
- L1: Digikey 732-1231-1-ND -> (none); Digikey Part Number (none) -> 732-1231-1-ND
- P1: Digikey Part Number (none) -> 900-1054440011CT-ND
- Q1: Digikey 785-1795-1-ND -> (none); Digikey Part Number (none) -> 785-1795-1-ND
- Q2, Q3, Q4, Q5: Digikey BSS214NH6327XTSA1CT-ND -> (none); Digikey Part Number (none) -> BSS214NH6327XTSA1CT-ND
- R1, R13, R15, R18, R2, R25: Digikey Part Number (none) -> A129689CT-ND; SPN A129689CT-ND -> (none)
- R14, R16, R17, R21: Digikey Part Number (none) -> 311-47KGRCT-ND; SPN 311-47KGRCT-ND -> (none)
- U1: Digikey Part Number (none) -> 497-17355-1-ND
- U2: Digikey Part Number (none) -> LM2596S-5.0/NOPB-ND
- U5: Digikey EG4938-ND -> (none); Digikey Part Number (none) -> EG4938-ND
- U6: Digikey Part Number (none) -> 296-DRV8220DRLRCT-ND
